Commit message: Corrected IMU name in amr_description package (urdf and meshes) and defined parameters for the imu with the xsens_params.yaml file.

File: src/amr_description/amr/urdf/amr.urdf (robot description, URDF)
Before this commit: robot Amr, 35 links, 34 joints
Links:
- removed link IMU_MTI_670_Link
- added link IMU_MTI_680g_Link, mass 0.224157079632679; collision mesh filename=package://amr_description/amr/meshes/IMU_MTI_680g_Link.STL; visual mesh filename=package://amr_description/amr/meshes/IMU_MTI_680g_Link.STL
Joints:
- removed joint IMU_MTI_670_Joint
- added joint IMU_MTI_680g_Joint: type fixed, parent Base_Link, child IMU_MTI_680g_Link, origin xyz=0 0 0.087925 rpy=0 0 0, axis 0 0 0
