Commit message: Make a customized sized world encircled by walls.

File: src/amr_simulation/worlds/world2.sdf.xacro (robot description, xacro)
@@ -1,6 +1,5 @@
 <?xml version="1.0"?>
 <sdf version="1.10" xmlns:xacro="http://www.ros.org/wiki/xacro">
-    <!-- A default function to include models -->
-    <xacro:macro name="include_model" params="name model pose">
+     <xacro:macro name="include_model" params="name model pose">
         <include>
         <name>${name}</name>
@@ -39,22 +38,11 @@
             <uri>https://fuel.gazebosim.org/1.0/OpenRobotics/models/Sun</uri>
         </include>
-        <!-- ++++++++++++++++++++++++++++++++++ Parameters +++++++++++++++++++++++++++++++++++++++++++++++++ -->
-        <xacro:property name="wall_width" value="5" />
-        <xacro:property name="wall_length" value="140" />
-        <xacro:property name="wall_height" value="5" />
-        <xacro:property name="x_size_floor" value="160" />
-        <xacro:property name="y_size_floor" value="150" />
-        <xacro:property name="wall_x_pose" value="${x_size_floor / 2 - wall_width / 2}" />
-        <xacro:property name="wall_y_pose" value="${y_size_floor / 2 - wall_width / 2}" />
-        <xacro:property name="wall_z_pose" value="${wall_height / 2}" />
-        <xacro:property name="wall_z_orientation" value="1.5708" />
         <!-- +++++++++++++++++++++++++++++++++Insert your models here++++++++++++++++++++++++++++++++++++ -->
         <!-- +++++++++++++++++++++++++++++++++++++++++++++++++++++++++++++++++++++++++++++++++++++++++++ -->
-        <xacro:include_model name="White floor" model="white_floor" pose="0 0 0 0 0 0"/>
-        <xacro:include_model name="Wall north" model="wall" pose="${wall_x_pose} 0 ${wall_z_pose} 0 0 0"/>
-        <xacro:include_model name="Wall east" model="wall" pose="0 ${wall_y_pose} ${wall_z_pose} 0 0 -${wall_z_orientation}"/>
-        <xacro:include_model name="Wall west" model="wall" pose="0 -${wall_y_pose} ${wall_z_pose} 0 0 ${wall_z_orientation}"/>
-        <xacro:include_model name="Wall south" model="wall" pose="-${wall_x_pose} 0 ${wall_z_pose} 0 0 0"/>
-        <xacro:include_model name="Obstacle Scenario" model="obstacle_scenario" pose="0 0 0 0 0 0"/>
+        <xacro:include filename="$(find amr_simulation)/models/white_floor/model.sdf.xacro" ns="my_white_floor"/>
+        <xacro:include filename="$(find amr_simulation)/scenarios/wall_fortress/model.sdf.xacro" ns="wall_fortress"/>
+        <xacro:my_white_floor.white_floor/>
+        <xacro:wall_fortress.wall_fortress/>
+        <!-- <xacro:include_model name="Obstacle Scenario" model="obstacle_scenario" pose="0 0 0 0 0 0"/>
         <xacro:include_model name="Obstacle Scenario2" model="obstacle_scenario" pose="30 0 0 0 0 0"/>
         <xacro:include_model name="Obstacle Scenario3" model="obstacle_scenario" pose="0 30 0 0 0 0"/>
@@ -66,5 +54,5 @@
         <xacro:include_model name="Obstacle Scenario9" model="obstacle_scenario" pose="25 -25 0 0 0 -10"/>
         <xacro:include_model name="Obstacle Scenario10" model="obstacle_scenario" pose="-25 25 0 0 0 10"/>
-        <xacro:include_model name="bluevehicleA" model="vehicle_blue" pose="2 4 0.05 0 0 0"/>
+        <xacro:include_model name="bluevehicleA" model="vehicle_blue" pose="2 4 0.05 0 0 0"/> -->
     </world>
 </sdf>
