Commit message: Change floor size; Add model with 4 wheels; Add joint_states to all wheels of x1;

File: src/amr_simulation/models/white_floor/model.sdf.xacro (robot description, xacro)
@@ -1,6 +1,6 @@
 <?xml version="1.0"?>
 <sdf version="1.10" xmlns:xacro="http://www.ros.org/wiki/xacro">
-    <xacro:property name="x_size_floor" value="100" />
-    <xacro:property name="y_size_floor" value="100" />
+    <xacro:property name="x_size_floor" value="150" />
+    <xacro:property name="y_size_floor" value="150" />
     <xacro:macro name="brown_floor">
         <model name="Brown Floor">
