Commit message: Change the simulation map so it looks closer to a corridor.

File: src/amr_simulation/models/white_floor/model.sdf.xacro (robot description, xacro)
@@ -1,6 +1,6 @@
 <?xml version="1.0"?>
 <sdf version="1.10" xmlns:xacro="http://www.ros.org/wiki/xacro">
-    <xacro:property name="x_size_floor" value="150" />
-    <xacro:property name="y_size_floor" value="150" />
+    <xacro:property name="x_size_floor" value="1000" />
+    <xacro:property name="y_size_floor" value="200" />
     <xacro:macro name="brown_floor">
         <model name="Brown Floor">

File: src/amr_simulation/worlds/world.sdf.xacro (robot description, xacro)
@@ -47,5 +47,5 @@
         <xacro:floor_namespace.brown_floor/>
         <xacro:wall_fortress_namespace.wall_fortress/>
-        <xacro:include_model name="Obstacle Scenario" model="obstacle_scenario" pose="0 0 0 0 0 0"/>
+        <!-- <xacro:include_model name="Obstacle Scenario" model="obstacle_scenario" pose="0 0 0 0 0 0"/>
         <xacro:include_model name="Obstacle Scenario2" model="obstacle_scenario" pose="30 0 0 0 0 0"/>
         <xacro:include_model name="Obstacle Scenario3" model="obstacle_scenario" pose="0 30 0 0 0 0"/>
@@ -56,5 +56,5 @@
         <xacro:include_model name="Obstacle Scenario8" model="obstacle_scenario" pose="-25 -25 0 0 0 10"/>
         <xacro:include_model name="Obstacle Scenario9" model="obstacle_scenario" pose="25 -25 0 0 0 -10"/>
-        <xacro:include_model name="Obstacle Scenario10" model="obstacle_scenario" pose="-25 25 0 0 0 10"/>
+        <xacro:include_model name="Obstacle Scenario10" model="obstacle_scenario" pose="-25 25 0 0 0 10"/> -->
         <!-- <xacro:include_model name="vehicle" model="vehicle_blue" pose="2 4 0.05 0 0 0"/> -->
     </world>
